Commit message: Working follow left implementation

File: robot_maze_solver/description/lidar.xacro (robot description, xacro)
@@ -4,5 +4,5 @@
         <parent link='chassis'/>
         <child link='lidar'/>
-        <origin xyz='0.75 0 0.255' rpy='0 0 0'/>
+        <origin xyz='0.250 0 0.255' rpy='0 0 0'/>
     </joint>
     <link name="lidar">

File: robot_maze_solver/description/robot_body.xacro (robot description, xacro)
@@ -14,5 +14,5 @@
     <link name="base_link"></link>
     <xacro:property name="width" value="0.5"/>
-    <xacro:property name="length" value="1.0"/>
+    <xacro:property name="length" value="0.5"/>
     <xacro:property name="height" value="0.25"/>
     <xacro:property name="wheel_radius" value="0.1"/>
